File: Hardware/Schematic/ActiveLoad.sch (KiCad schematic (older format))
At the start: 0 parts

Commit message: feat: added devices BTS117, LM9036M and STM32F072C8
Parts:
- added HS?: SK 129-50 STS, Heatsinks:Heatsink_Fischer_SK129-STS_42x25mm_2xDrill2.5mm, symbol HEATSINK
- added Q?: BTS117, TO-220, symbol BTS117
- added U?: STM32F072C8, LQFP48, symbol STM32F072CB
- added U? (x2): MCP6002, symbol MCP6002
Other:
- note added: "Use MCP6442 for better performance"
Changed lines of the file:
@@
 LIBS:contrib
 LIBS:valves
+LIBS:stm32f0
+LIBS:bts117
 LIBS:ActiveLoad-cache
 EELAYER 25 0
@@
 Comment4 ""
 $EndDescr
+$Comp
+L STM32F072CB U?
+U 1 1 569BF24D
+P 7100 4150
+F 0 "U?" H 5600 6050 60  0000 C CNN
+F 1 "STM32F072C8" H 8350 2250 60  0000 C CNN
+F 2 "LQFP48" H 7100 4150 40  0000 C CIN
+F 3 "" H 7100 4150 60  0000 C CNN
+	1    7100 4150
+	1    0    0    -1
+$EndComp
+$Comp
+L BTS117 Q?
+U 1 1 569BF4D2
+P 3350 1900
+F 0 "Q?" H 3550 1975 50  0000 L CNN
+F 1 "BTS117" H 3550 1900 50  0000 L CNN
+F 2 "TO-220" H 3550 1825 50  0000 L CIN
+F 3 "" H 3350 1900 50  0000 L CNN
+	1    3350 1900
+	1    0    0    -1
+$EndComp
+$Comp
+L MCP6002 U?
+U 1 1 569BF6A4
+P 10250 1900
+F 0 "U?" H 10250 2050 50  0000 L CNN
+F 1 "MCP6002" H 10250 1750 50  0000 L CNN
+F 2 "" H 10150 1950 50  0000 C CNN
+F 3 "" H 10250 2050 50  0000 C CNN
+	1    10250 1900
+	1    0    0    -1
+$EndComp
+$Comp
+L MCP6002 U?
+U 2 1 569BF725
+P 10350 2600
+F 0 "U?" H 10350 2750 50  0000 L CNN
+F 1 "MCP6002" H 10350 2450 50  0000 L CNN
+F 2 "" H 10250 2650 50  0000 C CNN
+F 3 "" H 10350 2750 50  0000 C CNN
+	2    10350 2600
+	1    0    0    -1
+$EndComp
+Text Notes 9600 1350 0    60   ~ 0
+Use MCP6442 for better performance
+$Comp
+L HEATSINK HS?
+U 1 1 569BF978
+P 3500 1300
+F 0 "HS?" H 3500 1500 50  0000 C CNN
+F 1 "SK 129-50 STS" H 3500 1250 50  0000 C CNN
+F 2 "Heatsinks:Heatsink_Fischer_SK129-STS_42x25mm_2xDrill2.5mm" H 3500 1300 50  0001 C CNN
+F 3 "" H 3500 1300 50  0000 C CNN
+	1    3500 1300
+	1    0    0    -1
+$EndComp
 $EndSCHEMATC

Commit message: updated schematic
Parts:
- added C? (x9): 100n, Capacitors_SMD:C_0603, symbol C
- added C?: 4n7/50V, Capacitors_SMD:C_1210, symbol C
- added C?: 10n, Capacitors_SMD:C_0603, symbol C
- added D?: Run LED green, LEDs:LED_0603, symbol LED
- added FB? (x2): 8,2µH/0805, Resistors_SMD:R_0805, symbol FILTER
- added P?: TC2030-CTX, Tag-Connect:TC2030_SMALL, symbol TC2030-CTX
- added P?: USB_B, symbol USB_B
- added R? (x4): 10k, Resistors_SMD:R_0603, symbol R
- added R?: 220, Resistors_SMD:R_0603, symbol R
- added R?: 1M, Resistors_SMD:R_1206, symbol R
- added R?: 0, Resistors_SMD:R_0603, symbol R
- added R?: 100, Resistors_SMD:R_0603, symbol R
- added R?: 100m, symbol R
- added R? (x2): 9k, Resistors_SMD:R_0603, symbol R
- added R? (x2): 1k, Resistors_SMD:R_0603, symbol R
- added SW?: FSMSM, Buttons_Switches_SMD:SW_SPST_FSMSM, symbol SW_PUSH
- added SW?: SWITCH_INV, symbol SWITCH_INV
- added U?: MAX3207E, symbol MAX3207E
- added U?: LM9036M, SO8, symbol LM9036M
- added X?: CSTCE8M00G15, ceralock:CSTCE_G15C, symbol RESONATOR
Connections:
- net +3V3: now reaches U?.1 (VBAT)
- net +3V3: now also U?.8 (V+), C?.1, C?.2, P?.1 (VCC), R?.1, SW?.1, U?.5 (VCC)
- net at U?.10 (WKUP1/RTC_TAMP2/ADC_IN0/TIM2_CH1_ETR/USART4_TX/PA0): now also C?.1, R?.1
- net at U?.14 (SPI1_NSS/I2S1_WS/ADC_IN4/TIM14_CH1/USART2_CK/DAC1/PA4): now also R?.1
- net GND: now reaches U?.23 (VSS)
- net GND: now also U?.35 (VSS), U?.47 (VSS), C?.1, C?.2, C?.2, C?.2, D?.1 (K), FB?.2, P?.5 (GND), R?.1, R?.1, U?.2 (GND), X?.2
- net at U?.24 (VDD): now also U?.36 (VDD2), U?.48 (VDD)
- net USB_D-: now reaches U?.32 (CAN_RX/USART1_CTS/TIM1_CH4/USB_DM/EVENTOUT/PA11)
- net USB_D-: now also P?.2 (D-), U?.1 (I/O1)
- net USB_D+: now reaches U?.33 (CAN_TX/USART1_RTS/TIM1_ETR/USB_DP/EVENTOUT/PA12)
- net USB_D+: now also P?.3 (D+), U?.4 (I/O2)
- net SWDIO: now reaches U?.34 (IR_OUT/SWDAT/USB_NOE/PA13)
- net SWDIO: now also P?.2 (SWDIO/TMS)
- net SWCLK: now reaches U?.37 (USART2_TX/SWCLK/PA14)
- net SWCLK: now also P?.4 (SWCLK/TCK)
- net at U?.44 (BOOT0): now also R?.2, SW?.2
- net at U?.5 (PF0/OSC_IN): now also X?.1
- net at U?.6 (PF1/OSC_OUT): now also X?.3
- net NRST: now reaches U?.7 (~NRST)
- net NRST: now also C?.1, P?.3 (~RESET~), R?.2
- net GNDA: now reaches U?.8 (VSSA)
- net GNDA: now also U?.4 (V-), C?.2, C?.2, C?.2, R?.2, R?.2, R?.2
- net +3.3VADC: now reaches U?.9 (VDDA)
- net at Q?.1 (G): now also R?.2
- net VCC: now reaches Q?.2 (D)
- net VCC: now also SW?.3
- net at Q?.3 (S): now also R?.1, R?.2
- net at U?.1: now also R?.1, R?.1
- net at U?.2 (-): now also U?.5 (+), C?.2, R?.1
- net at U?.3 (+): now also C?.1, R?.1, R?.2
- net at U?.6 (-): now also R?.1, R?.2
- net at U?.7: now also R?.1, R?.2
- new net: D?.2 (A), R?.2
- new net: FB?.1, P?.1 (VCC)
- new net: FB?.1, P?.4 (GND)
- new net: C?.1, P?.5 (shield), R?.2
- new net: C?.1, R?.2
- new net +5V: C?.1, FB?.2, SW?.1
- no-connect marks 0 -> 1
Other:
- note added: "0,1 mV/mA"
- note added: "Bootloader"
- note added: "Gain: 0,1"
- note added: "Gain: 10"
- note added: "Mini USB"
- note added: "TBD: UARTx TX"
- moved on the sheet: HS?, Q?, U?, U?A, U?B

Commit message: updated schematic added DOG display library
Parts:
- added C?: 100n/50V, Capacitors_SMD:C_0805, symbol C
- added C?: 47u/16V, symbol CP
- added C?: 4u7/16V, Capacitors_SMD:C_0805, symbol C
- added C?: 4u7/50V, Capacitors_SMD:C_1206, symbol C
- added C? (x2): 4u7, Capacitors_SMD:C_0805, symbol C
- added C?: 100n, Capacitors_SMD:C_0603, symbol C
- added C? (x3): 1u, Capacitors_SMD:C_0603, symbol C
- added C? (x3): 10n, Capacitors_SMD:C_0603, symbol C
- added E?: STEC12E08, symbol Encoder_switch
- added FB?: 8,2µH/0805, Resistors_SMD:R_0805, symbol FILTER
- added JP? (x2): Jumper_NC_Small, symbol Jumper_NC_Small
- added LCD?: EA-DOGS104-A, symbol EA-DOGS104-A
- added R? (x3): 10k, Resistors_SMD:R_0603, symbol R
- U?: value LM9036M -> LM9036M-3.3
Connections:
- net labels added: GNDPWR
- wire segments 142 -> 201
Other:
- note added: "0.3R ≤ ESR ≤ 8R"
- moved on the sheet: C?, D?, HS?, Q?, R?, SW?, U?, U?A, U?B

Commit message: updated schematic
Parts:
- removed E?: STEC12E08, symbol Encoder_switch
- added C?: 100n, Capacitors_SMD:C_0603, symbol C
- added ENC?: ALPS-STEC12E08, ALPS-STEC12E08:ALPS-STEC12E08, symbol ALPS-STEC12E08
- added P?: AKL 101-2, w_conn_screw:mors_2p, symbol CONN_01X02
- added P?: Banana jacks, Connect:Banana_Jack_2Pin, symbol CONN_01X02
- added R? (x2): 10k, Resistors_SMD:R_0603, symbol R
- added U?: DS18B20, TO_SOT_Packages_THT:TO-92_Inline_Narrow_Oval, symbol DS18B20
- P?: footprint (none) -> Connect:USB_Mini-B
- SW?: value SWITCH_INV -> ESP4020; footprint (none) -> ece_switches:ESP40XX
- U?: footprint LQFP48 -> Housings_QFP:LQFP-48_7x7mm_Pitch0.5mm
- U? (x2): footprint (none) -> Housings_SOIC:SOIC-8_3.9x4.9mm_Pitch1.27mm
- U?: footprint (none) -> TO_SOT_Packages_SMD:SOT-23-6
- U?: footprint SO8 -> Housings_SOIC:SOIC-8_3.9x4.9mm_Pitch1.27mm
Connections:
- net labels added: ENC_A, ENC_B, ENC_SW, TEMP
- wire segments 201 -> 228
Other:
- note added: "Screw terminal"
- note added: "TBD"
- note added: "TBD: Shunt package"
- note added: "Thermally connect\nsensor to FET!"
- moved on the sheet: C?, HS?, P?, R?

Commit message: (nearly) finished schematic
Parts:
- added R16: 390, Resistors_SMD:R_0603, symbol R
- added R17, R20: 100m, Resistors_SMD:R_2512, symbol R
- added R18: 240, Resistors_SMD:R_0603, symbol R
- added U5: LM317AEMP, TO_SOT_Packages_SMD:SOT-223, symbol LM317AEMP
- C25: renamed from C?; footprint (none) -> Capacitors_SMD:c_elec_6.3x5.3
- JP1, JP2: renamed from JP?; footprint (none) -> Oddities:NetTie-I_Connected_SMD
- LCD1: renamed from LCD?; footprint (none) -> dog-displays:DOGS104
- Q1: renamed from Q?; footprint TO-220 -> TO_SOT_Packages_THT:TO-220_Neutral123_Vertical
- R19: renamed from R?; footprint (none) -> Resistors_ThroughHole:Resistor_Cement_Horizontal_Meggitt-SBC-2
- gave numbers to parts that had none: 59
Connections:
- net +3V3: now also R18.2, U5.2 (OUT)
- net GND: now also R16.2
- net GNDPWR: now also R17.2, R20.2
- net at Q1.3 (S), R15.2, R19.1: now also R17.1, R20.1
- net at R13.1, R14.1: now also U4.7; no longer U4.1
- net at C21.2, R15.1: now also U4.3 (+), U4.6 (-); no longer U4.2 (-), U4.5 (+)
- net at C18.1, R11.1, R8.2: now also U4.5 (+); no longer U4.3 (+)
- net at R10.2, R12.1: now also U4.2 (-); no longer U4.6 (-)
- net at R10.1, R9.2: now also U4.1; no longer U4.7
- net at C22.1, SW2.2, U6.8 (VIN): now also U5.3 (IN)
- new net: R16.1, R18.1, U5.1 (ADJ)
- no-connect marks 1 -> 22
Other:
- note added: "Alternative regulator\nFit EITHER U5 or U6"
- note added: "Different shunt packages\nSelect as desired"
- note added: "Thermally connect\nU3 to FET!"
- note removed: "TBD: Shunt package"
- note removed: "Thermally connect\nsensor to FET!"
- moved on the sheet: R14, R15

Commit message: finished schematic
Parts:
- added R23, R24, R25, R26: 0, Resistors_SMD:R_0603, symbol R
- R10: value 9k -> 18k
- R12: value 1k -> 2k
- R8: value 9k -> 10k
- R9: value 10k -> 1k
Connections:
- net +3V3: now also R25.2, R26.2; no longer R18.2, U5.2 (OUT), U6.1 (VOUT)
- net GND: no longer P2.2 (P2), P3.2 (P2)
- net GNDA: now also JP1.1; no longer JP1.2, JP2.1
- net GNDPWR: now also JP1.2, JP2.1, P2.2 (P2), P3.2 (P2); no longer JP1.1
- net at C18.1, R11.1, R8.2: now also U4.3 (+); no longer U4.5 (+)
- net at C21.2, R15.1: now also U4.2 (-), U4.5 (+); no longer U4.3 (+), U4.6 (-)
- net at R13.1, R14.1: now also U4.1; no longer U4.7
- net at R10.1, R9.2: now also U4.7; no longer U4.1
- net at R10.2, R12.1: now also U4.6 (-); no longer U4.2 (-)
- net at C22.1, SW2.2: now also R23.2, R24.1; no longer U5.3 (IN), U6.8 (VIN)
- new net: R26.1, U6.1 (VOUT)
- new net: R24.2, U6.8 (VIN)
- new net: R18.2, R25.1, U5.2 (OUT)
- new net: R23.1, U5.3 (IN)
Other:
- note added: "Power supply select"
- note removed: "0.3R ≤ ESR ≤ 8R"
- moved on the sheet: C25
Changed lines of the file:
@@
 $Comp
 L MCP6002 U4
-U 2 1 569BF6A4
+U 1 1 569BF6A4
 P 8250 1250
 F 0 "U4" H 8250 1400 50  0000 L CNN
@@
 F 2 "Housings_SOIC:SOIC-8_3.9x4.9mm_Pitch1.27mm" H 8150 1300 50  0001 C CNN
 F 3 "" H 8250 1400 50  0000 C CNN
-	2    8250 1250
+	1    8250 1250
 	1    0    0    -1
 $EndComp
 $Comp
 L MCP6002 U4
-U 1 1 569BF725
+U 2 1 569BF725
 P 7500 2300
 F 0 "U4" H 7500 2450 50  0000 L CNN
@@
 F 2 "Housings_SOIC:SOIC-8_3.9x4.9mm_Pitch1.27mm" H 7400 2350 50  0001 C CNN
 F 3 "" H 7500 2450 50  0000 C CNN
-	1    7500 2300
+	2    7500 2300
 	-1   0    0    -1
 $EndComp
@@
 L GNDA #PWR022
 U 1 1 56AE02E9
-P 10600 6250
-F 0 "#PWR022" H 10600 6000 50  0001 C CNN
-F 1 "GNDA" H 10600 6100 50  0000 C CNN
-F 2 "" H 10600 6250 50  0000 C CNN
-F 3 "" H 10600 6250 50  0000 C CNN
-	1    10600 6250
+P 10200 6250
+F 0 "#PWR022" H 10200 6000 50  0001 C CNN
+F 1 "GNDA" H 10200 6100 50  0000 C CNN
+F 2 "" H 10200 6250 50  0000 C CNN
+F 3 "" H 10200 6250 50  0000 C CNN
+	1    10200 6250
 	1    0    0    -1
 $EndComp
@@
 P 6900 1150
 F 0 "R8" V 6980 1150 50  0000 C CNN
-F 1 "9k" V 6900 1150 50  0000 C CNN
+F 1 "10k" V 6900 1150 50  0000 C CNN
 F 2 "Resistors_SMD:R_0603" V 6830 1150 50  0001 C CNN
 F 3 "" H 6900 1150 50  0000 C CNN
@@
 P 6900 2650
 F 0 "R9" V 6980 2650 50  0000 C CNN
-F 1 "10k" V 6900 2650 50  0000 C CNN
+F 1 "1k" V 6900 2650 50  0000 C CNN
 F 2 "Resistors_SMD:R_0603" V 6830 2650 50  0001 C CNN
 F 3 "" H 6900 2650 50  0000 C CNN
@@
 P 7600 2850
 F 0 "R10" V 7680 2850 50  0000 C CNN
-F 1 "9k" V 7600 2850 50  0000 C CNN
+F 1 "18k" V 7600 2850 50  0000 C CNN
 F 2 "Resistors_SMD:R_0603" V 7530 2850 50  0001 C CNN
 F 3 "" H 7600 2850 50  0000 C CNN
@@
 P 8150 2850
 F 0 "R12" V 8230 2850 50  0000 C CNN
-F 1 "1k" V 8150 2850 50  0000 C CNN
+F 1 "2k" V 8150 2850 50  0000 C CNN
 F 2 "Resistors_SMD:R_0603" V 8080 2850 50  0001 C CNN
 F 3 "" H 8150 2850 50  0000 C CNN
@@
 L CP C25
 U 1 1 56B124E4
-P 10700 5450
-F 0 "C25" H 10725 5550 50  0000 L CNN
-F 1 "47u/16V" H 10725 5350 50  0000 L CNN
-F 2 "Capacitors_SMD:c_elec_6.3x5.3" H 10738 5300 50  0001 C CNN
-F 3 "" H 10700 5450 50  0000 C CNN
-	1    10700 5450
+P 10800 5450
+F 0 "C25" H 10825 5550 50  0000 L CNN
+F 1 "47u/16V" H 10825 5350 50  0000 L CNN
+F 2 "Capacitors_SMD:c_elec_6.3x5.3" H 10838 5300 50  0001 C CNN
+F 3 "" H 10800 5450 50  0000 C CNN
+	1    10800 5450
 	1    0    0    -1
 $EndComp
@@
 L +3.3V #PWR030
 U 1 1 56B12A9E
-P 10700 5050
-F 0 "#PWR030" H 10700 4900 50  0001 C CNN
-F 1 "+3.3V" H 10700 5190 50  0000 C CNN
-F 2 "" H 10700 5050 50  0000 C CNN
-F 3 "" H 10700 5050 50  0000 C CNN
-	1    10700 5050
+P 10800 4850
+F 0 "#PWR030" H 10800 4700 50  0001 C CNN
+F 1 "+3.3V" H 10800 4990 50  0000 C CNN
+F 2 "" H 10800 4850 50  0000 C CNN
+F 3 "" H 10800 4850 50  0000 C CNN
+	1    10800 4850
 	1    0    0    -1
 $EndComp
@@
 	1    0    0    -1
 $EndComp
-Text Notes 11150 5900 1    60   ~ 0
-0.3R ≤ ESR ≤ 8R
 $Comp
 L C C19
@@
 L GNDPWR #PWR035
 U 1 1 56B1EA57
-P 10200 6250
-F 0 "#PWR035" H 10200 6050 50  0001 C CNN
-F 1 "GNDPWR" H 10200 6120 50  0000 C CNN
-F 2 "" H 10200 6200 50  0000 C CNN
-F 3 "" H 10200 6200 50  0000 C CNN
-	1    10200 6250
+P 10600 6250
+F 0 "#PWR035" H 10600 6050 50  0001 C CNN
+F 1 "GNDPWR" H 10600 6120 50  0000 C CNN
+F 2 "" H 10600 6200 50  0000 C CNN
+F 3 "" H 10600 6200 50  0000 C CNN
+	1    10600 6250
 	1    0    0    -1
 $EndComp
@@
 $EndComp
 $Comp
-L GND #PWR048
-U 1 1 56B4EC9F
-P 850 5800
-F 0 "#PWR048" H 850 5550 50  0001 C CNN
-F 1 "GND" H 850 5650 50  0000 C CNN
-F 2 "" H 850 5800 50  0000 C CNN
-F 3 "" H 850 5800 50  0000 C CNN
-	1    850  5800
-	1    0    0    -1
-$EndComp
-$Comp
 L CONN_01X02 P3
 U 1 1 56B537EB
@@
 $EndComp
 $Comp
-L +3.3V #PWR049
+L +3.3V #PWR048
 U 1 1 56B57D9B
 P 5550 900
-F 0 "#PWR049" H 5550 750 50  0001 C CNN
+F 0 "#PWR048" H 5550 750 50  0001 C CNN
 F 1 "+3.3V" H 5550 1040 50  0000 C CNN
 F 2 "" H 5550 900 50  0000 C CNN
@@
 $EndComp
 $Comp
-L GND #PWR050
+L GND #PWR049
 U 1 1 56B58A58
 P 5550 1600
-F 0 "#PWR050" H 5550 1350 50  0001 C CNN
+F 0 "#PWR049" H 5550 1350 50  0001 C CNN
 F 1 "GND" H 5550 1450 50  0000 C CNN
 F 2 "" H 5550 1600 50  0000 C CNN
@@
 $EndComp
 $Comp
-L GND #PWR051
+L GND #PWR050
 U 1 1 56B59B6C
 P 6250 950
-F 0 "#PWR051" H 6250 700 50  0001 C CNN
+F 0 "#PWR050" H 6250 700 50  0001 C CNN
 F 1 "GND" H 6250 800 50  0000 C CNN
 F 2 "" H 6250 950 50  0000 C CNN
@@
 	7200 4950 7200 5400
 Wire Wire Line
-	8750 5200 9350 5200
-Wire Wire Line
-	8850 4100 8850 5350
-Wire Wire Line
 	8850 5650 8850 5900
 Wire Wire Line
@@
 	9300 5850 9300 5450
 Wire Wire Line
-	7200 5850 10700 5850
+	7200 5850 10800 5850
 Connection ~ 8850 5850
 Wire Wire Line
@@
 Connection ~ 10450 5550
 Wire Wire Line
-	10700 5850 10700 5600
+	10800 5850 10800 5600
 Connection ~ 10450 5850
 Wire Wire Line
-	10700 5050 10700 5300
-Wire Wire Line
-	10350 5200 10700 5200
-Connection ~ 10700 5200
+	10800 4850 10800 5300
+Connection ~ 10800 5200
 Connection ~ 8850 5200
 Wire Wire Line
@@
 Wire Wire Line
 	9800 4100 9800 4900
-Wire Wire Line
-	9800 4900 10450 4900
-Wire Wire Line
-	10450 4900 10450 5200
-Connection ~ 10450 5200
 $Comp
 L R R18
@@
 $EndComp
 $Comp
-L GND #PWR052
+L GND #PWR051
 U 1 1 56B3BC22
 P 9300 4900
-F 0 "#PWR052" H 9300 4650 50  0001 C CNN
+F 0 "#PWR051" H 9300 4650 50  0001 C CNN
 F 1 "GND" H 9300 4750 50  0000 C CNN
 F 2 "" H 9300 4900 50  0000 C CNN
@@
 NoConn ~ 5650 5850
 NoConn ~ 5650 4650
+$Comp
+L R R24
+U 1 1 56B5247C
+P 9100 5200
+F 0 "R24" V 9180 5200 50  0000 C CNN
+F 1 "0" V 9100 5200 50  0000 C CNN
+F 2 "Resistors_SMD:R_0603" V 9030 5200 50  0001 C CNN
+F 3 "" H 9100 5200 50  0000 C CNN
+	1    9100 5200
+	0    -1   -1   0
+$EndComp
+Wire Wire Line
+	8750 5200 8950 5200
+Wire Wire Line
+	9250 5200 9350 5200
+$Comp
+L R R23
+U 1 1 56B54167
+P 8850 4700
+F 0 "R23" V 8930 4700 50  0000 C CNN
+F 1 "0" V 8850 4700 50  0000 C CNN
+F 2 "Resistors_SMD:R_0603" V 8780 4700 50  0001 C CNN
+F 3 "" H 8850 4700 50  0000 C CNN
+	1    8850 4700
+	1    0    0    -1
+$EndComp
+Wire Wire Line
+	8850 4850 8850 5350
+Wire Wire Line
+	8850 4100 8850 4550
+$Comp
+L R R25
+U 1 1 56B55C72
+P 10550 4900
+F 0 "R25" V 10630 4900 50  0000 C CNN
+F 1 "0" V 10550 4900 50  0000 C CNN
+F 2 "Resistors_SMD:R_0603" V 10480 4900 50  0001 C CNN
+F 3 "" H 10550 4900 50  0000 C CNN
+	1    10550 4900
+	0    -1   -1   0
+$EndComp
+Wire Wire Line
+	9800 4900 10400 4900
+$Comp
+L R R26
+U 1 1 56B565C7
+P 10550 5200
+F 0 "R26" V 10630 5200 50  0000 C CNN
+F 1 "0" V 10550 5200 50  0000 C CNN
+F 2 "Resistors_SMD:R_0603" V 10480 5200 50  0001 C CNN
+F 3 "" H 10550 5200 50  0000 C CNN
+	1    10550 5200
+	0    -1   -1   0
+$EndComp
+Wire Wire Line
+	10350 5200 10400 5200
+Wire Wire Line
+	10700 5200 10800 5200
+Wire Wire Line
+	10700 4900 10800 4900
+Connection ~ 10800 4900
+Text Notes 7850 4950 0    60   ~ 0
+Power supply select
+$Comp
+L GNDPWR #PWR052
+U 1 1 56B6513B
+P 850 5800
+F 0 "#PWR052" H 850 5600 50  0001 C CNN
+F 1 "GNDPWR" H 850 5670 50  0000 C CNN
+F 2 "" H 850 5750 50  0000 C CNN
+F 3 "" H 850 5750 50  0000 C CNN
+	1    850  5800
+	1    0    0    -1
+$EndComp
 $EndSCHEMATC
