File: Hardware/Schematic/ActiveLoad.sch (KiCad schematic (older format))
At the start: 75 parts, among them P1 USB_OTG, P2 Banana jacks, P3 AKL 101-2, P4 TC2030-CTX, Q1 BTS117, SW1 FSMSM, SW2 ESP4020, U1 MAX3207E, U2 STM32F072C8, U3 DS18B20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

Commit message: updated schematic and PCB (added VSENSE)
Parts:
- added D2: BAS40, TO_SOT_Packages_SMD:SOT-23, symbol BAS40
- added R27: 56k, Resistors_SMD:R_0603, symbol R
- added R28: 4k7, Resistors_SMD:R_0603, symbol R
Connections:
- net +3.3VADC: now also D2.3 (K)
- net GND: now also R28.2
- net VCC: now also R27.1
- net VSENSE: now reaches U2.13 (USART2_RX/ADC1_IN3/TIM2_CH4/PA3)
- net VSENSE: now also D2.1 (A), R27.2, R28.1
- no-connect marks 18 -> 17
Other:
- moved on the sheet: SW1
Changed lines of the file:
@@
 LIBS:ALPS-STEC12E08
 LIBS:maxim
+LIBS:bas40
 LIBS:ActiveLoad-cache
 EELAYER 25 0
@@
 L SW_PUSH SW1
 U 1 1 56A480F5
-P 1350 3600
-F 0 "SW1" H 1500 3710 50  0000 C CNN
-F 1 "FSMSM" H 1350 3520 50  0000 C CNN
-F 2 "Buttons_Switches_SMD:SW_SPST_FSMSM" H 1350 3600 50  0001 C CNN
-F 3 "" H 1350 3600 50  0000 C CNN
-	1    1350 3600
+P 1500 3600
+F 0 "SW1" H 1650 3710 50  0000 C CNN
+F 1 "FSMSM" H 1500 3520 50  0000 C CNN
+F 2 "Buttons_Switches_SMD:SW_SPST_FSMSM" H 1500 3600 50  0001 C CNN
+F 3 "" H 1500 3600 50  0000 C CNN
+	1    1500 3600
 	1    0    0    -1
 $EndComp
@@
 	0    -1   -1   0
 $EndComp
-Text Notes 1100 3850 0    60   ~ 0
+Text Notes 1450 3850 0    60   ~ 0
 Bootloader
 $Comp
@@
 L VCC #PWR047
 U 1 1 56B4DD93
-P 650 4950
-F 0 "#PWR047" H 650 4800 50  0001 C CNN
-F 1 "VCC" H 650 5100 50  0000 C CNN
-F 2 "" H 650 4950 50  0000 C CNN
-F 3 "" H 650 4950 50  0000 C CNN
-	1    650  4950
+P 650 4100
+F 0 "#PWR047" H 650 3950 50  0001 C CNN
+F 1 "VCC" H 650 4250 50  0000 C CNN
+F 2 "" H 650 4100 50  0000 C CNN
+F 3 "" H 650 4100 50  0000 C CNN
+	1    650  4100
 	1    0    0    -1
 $EndComp
@@
 	1400 3300 1250 3300
 Wire Wire Line
-	1650 3600 1850 3600
+	1800 3600 1850 3600
 Wire Wire Line
 	1850 3600 1850 3300
 Connection ~ 1850 3300
 Wire Wire Line
-	1050 3600 950  3600
+	950  3600 1200 3600
 Wire Wire Line
 	8150 1550 8150 1600
@@
 	9100 1600 9000 1600
 Wire Wire Line
-	9000 2200 9000 1600
-Wire Wire Line
-	7800 2200 9000 2200
+	9000 1600 9000 2200
+Wire Wire Line
+	9000 2200 7800 2200
 Wire Wire Line
 	8750 1350 8750 1250
@@
 	1000 6650 1000 6800
 Wire Wire Line
-	1100 6750 1100 6800
-Wire Wire Line
-	850  6750 1100 6750
+	1100 6800 1100 6750
+Wire Wire Line
+	1100 6750 850  6750
 Connection ~ 1000 6750
 Wire Wire Line
@@
 	650  5600 1000 5600
 Wire Wire Line
-	650  4950 650  5600
+	650  4100 650  5600
 Wire Wire Line
 	1000 5100 650  5100
@@
 NoConn ~ 2250 5550
 NoConn ~ 5650 3250
-NoConn ~ 5650 3450
 NoConn ~ 5650 3950
 NoConn ~ 5650 4050
@@
 Wire Wire Line
 	5650 5450 5850 5450
+Text GLabel 6050 3450 2    47   Input ~ 0
+VSENSE
+Wire Wire Line
+	6050 3450 5650 3450
+Text GLabel 1700 4300 2    47   Output ~ 0
+VSENSE
+$Comp
+L R R27
+U 1 1 56B81805
+P 900 4300
+F 0 "R27" V 980 4300 50  0000 C CNN
+F 1 "56k" V 900 4300 50  0000 C CNN
+F 2 "Resistors_SMD:R_0603" V 830 4300 50  0001 C CNN
+F 3 "" H 900 4300 50  0000 C CNN
+	1    900  4300
+	0    -1   -1   0
+$EndComp
+$Comp
+L R R28
+U 1 1 56B825E6
+P 1150 4500
+F 0 "R28" V 1230 4500 50  0000 C CNN
+F 1 "4k7" V 1150 4500 50  0000 C CNN
+F 2 "Resistors_SMD:R_0603" V 1080 4500 50  0001 C CNN
+F 3 "" H 1150 4500 50  0000 C CNN
+	1    1150 4500
+	1    0    0    -1
+$EndComp
+Wire Wire Line
+	750  4300 650  4300
+Connection ~ 650  4300
+Wire Wire Line
+	1050 4300 1700 4300
+Wire Wire Line
+	1150 4200 1150 4350
+Connection ~ 1150 4300
+Wire Wire Line
+	1150 4650 1150 4750
+$Comp
+L BAS40 D2
+U 1 1 56B83748
+P 1150 4050
+F 0 "D2" H 1150 4150 50  0000 C CNN
+F 1 "BAS40" H 1150 3950 50  0000 C CNN
+F 2 "TO_SOT_Packages_SMD:SOT-23" H 1150 4050 60  0001 C CNN
+F 3 "" H 1150 4050 60  0000 C CNN
+	1    1150 4050
+	0    1    1    0
+$EndComp
+$Comp
+L GND #PWR054
+U 1 1 56B87C49
+P 1150 4750
+F 0 "#PWR054" H 1150 4500 50  0001 C CNN
+F 1 "GND" H 1150 4600 50  0000 C CNN
+F 2 "" H 1150 4750 50  0000 C CNN
+F 3 "" H 1150 4750 50  0000 C CNN
+	1    1150 4750
+	1    0    0    -1
+$EndComp
+$Comp
+L +3.3VADC #PWR055
+U 1 1 56B88C20
+P 1150 3850
+F 0 "#PWR055" H 1300 3800 50  0001 C CNN
+F 1 "+3.3VADC" H 1150 3950 50  0000 C CNN
+F 2 "" H 1150 3850 50  0000 C CNN
+F 3 "" H 1150 3850 50  0000 C CNN
+	1    1150 3850
+	1    0    0    -1
+$EndComp
+Wire Wire Line
+	1150 3850 1150 3900
 $EndSCHEMATC

Commit message: fix: changed R8 and R11 to 18k and 2k to get a gain of 0,1
Parts:
- R11: value 1k -> 2k
- R8: value 10k -> 18k
Changed lines of the file:
@@
 P 6900 1150
 F 0 "R8" V 6980 1150 50  0000 C CNN
-F 1 "10k" V 6900 1150 50  0000 C CNN
+F 1 "18k" V 6900 1150 50  0000 C CNN
 F 2 "Resistors_SMD:R_0603" V 6830 1150 50  0001 C CNN
 F 3 "" H 6900 1150 50  0000 C CNN
@@
 P 7700 1450
 F 0 "R11" V 7780 1450 50  0000 C CNN
-F 1 "1k" V 7700 1450 50  0000 C CNN
+F 1 "2k" V 7700 1450 50  0000 C CNN
 F 2 "Resistors_SMD:R_0603" V 7630 1450 50  0001 C CNN
 F 3 "" H 7700 1450 50  0000 C CNN

Commit message: refactor: use MCP6002 (and not MCP6442 which does NOT have a better performance) fix: replaced 8,2µH/0805 inductors with BLM21PG331 EMI ferrite filters
Parts:
- C19: value 4u7/16V -> 4u7
- FB1, FB2, FB3: value 8,2µH/0805 -> BLM21PG331
Other:
- note removed: "Use MCP6442 for better performance"
Changed lines of the file:
@@
 	-1   0    0    -1
 $EndComp
-Text Notes 7900 2400 0    60   ~ 0
-Use MCP6442 for better performance
 $Comp
 L HEATSINK HS1
@@
 P 1600 1950
 F 0 "FB1" H 1600 2100 50  0000 C CNN
-F 1 "8,2µH/0805" H 1600 1850 50  0000 C CNN
+F 1 "BLM21PG331" H 1600 1850 50  0000 C CNN
 F 2 "Resistors_SMD:R_0805" H 1600 1950 50  0001 C CNN
 F 3 "" H 1600 1950 50  0000 C CNN
@@
 P 1850 1000
 F 0 "FB2" H 1850 1150 50  0000 C CNN
-F 1 "8,2µH/0805" H 1850 900 50  0000 C CNN
+F 1 "BLM21PG331" H 1850 900 50  0000 C CNN
 F 2 "Resistors_SMD:R_0805" H 1850 1000 50  0001 C CNN
 F 3 "" H 1850 1000 50  0000 C CNN
@@
 P 5100 2150
 F 0 "FB3" H 5100 2300 50  0000 C CNN
-F 1 "8,2µH/0805" H 5100 2050 50  0000 C CNN
+F 1 "BLM21PG331" H 5100 2050 50  0000 C CNN
 F 2 "Resistors_SMD:R_0805" H 5100 2150 50  0001 C CNN
 F 3 "" H 5100 2150 50  0000 C CNN
@@
 P 7650 5550
 F 0 "C19" H 7675 5650 50  0000 L CNN
-F 1 "4u7/16V" H 7675 5450 50  0000 L CNN
+F 1 "4u7" H 7675 5450 50  0000 L CNN
 F 2 "Capacitors_SMD:C_0805" H 7688 5400 50  0001 C CNN
 F 3 "" H 7650 5550 50  0000 C CNN

Commit message: fix: due to internal resistance of unbuffered DAC output (~15k), R8 is lowered to 2k
Parts:
- R8: value 18k -> 2k
Other:
- note added: "Gain: around 0,1\n(DAC has R_out of around 15k)"
- note removed: "Gain: 0,1"
Changed lines of the file:
@@
 P 6900 1150
 F 0 "R8" V 6980 1150 50  0000 C CNN
-F 1 "18k" V 6900 1150 50  0000 C CNN
+F 1 "2k" V 6900 1150 50  0000 C CNN
 F 2 "Resistors_SMD:R_0603" V 6830 1150 50  0001 C CNN
 F 3 "" H 6900 1150 50  0000 C CNN
@@
 	1    0    0    -1
 $EndComp
-Text Notes 7150 1050 0    60   ~ 0
-Gain: 0,1
+Text Notes 6550 1000 0    60   ~ 0
+Gain: around 0,1\n(DAC has R_out of around 15k)
 Text GLabel 3900 1000 2    47   BiDi ~ 0
 USB_D-

Commit message: doc: added note that LM317 has no reverse polarity protection
Other:
- note added: "If U5 is fitted, there is no\nreverse polarity protection!"
Changed lines of the file:
@@
 Wire Wire Line
 	1150 3850 1150 3900
+Text Notes 7600 6350 0    60   ~ 12
+If U5 is fitted, there is no\nreverse polarity protection!
 $EndSCHEMATC

Commit message: chore: change some resistors, caps and resonator to "DNF"
Parts:
- C5, C7: value 10n -> DNF
- R5, R6: value 10k -> DNF
Other:
- note added: "Do not fit"
Changed lines of the file:
@@
 P 3150 6950
 F 0 "R5" V 3230 6950 50  0000 C CNN
-F 1 "10k" V 3150 6950 50  0000 C CNN
+F 1 "DNF" V 3150 6950 50  0000 C CNN
 F 2 "Resistors_SMD:R_0603" V 3080 6950 50  0001 C CNN
 F 3 "" H 3150 6950 50  0000 C CNN
@@
 P 2350 7400
 F 0 "C5" H 2375 7500 50  0000 L CNN
-F 1 "10n" H 2375 7300 50  0000 L CNN
+F 1 "DNF" H 2375 7300 50  0000 L CNN
 F 2 "Capacitors_SMD:C_0603" H 2388 7250 50  0001 C CNN
 F 3 "" H 2350 7400 50  0000 C CNN
@@
 P 2600 7400
 F 0 "C7" H 2625 7500 50  0000 L CNN
-F 1 "10n" H 2625 7300 50  0000 L CNN
+F 1 "DNF" H 2625 7300 50  0000 L CNN
 F 2 "Capacitors_SMD:C_0603" H 2638 7250 50  0001 C CNN
 F 3 "" H 2600 7400 50  0000 C CNN
@@
 P 3150 7450
 F 0 "R6" V 3230 7450 50  0000 C CNN
-F 1 "10k" V 3150 7450 50  0000 C CNN
+F 1 "DNF" V 3150 7450 50  0000 C CNN
 F 2 "Resistors_SMD:R_0603" V 3080 7450 50  0001 C CNN
 F 3 "" H 3150 7450 50  0000 C CNN
@@
 Text Notes 7600 6350 0    60   ~ 12
 If U5 is fitted, there is no\nreverse polarity protection!
+Text Notes 1800 4550 0    60   ~ 12
+Do not fit
 $EndSCHEMATC
