File: Hardware/Schematic/ActiveLoad.kicad_pcb (KiCad board)
At the start: 2 copper layers, 50 x 100 mm, 83 parts, among them P1 USB_OTG, P2 Banana jacks, P3 AKL 101-2, P4 TC2030-CTX, Q1 BTS117, SW1 FSMSM, SW2 ESP4020, U1 MAX3207E, U2 STM32F072C8, U3 DS18B20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

Commit message: fix: changed R8 and R11 to 18k and 2k to get a gain of 0,1
Parts:
- R11: value 1k -> 2k
- R8: value 10k -> 18k
Changed lines of the file:
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@@
       (effects (font (size 1 1) (thickness 0.15)) (justify mirror))
     )
-    (fp_text value 10k (at 0 -1.9) (layer B.Fab)
+    (fp_text value 18k (at 0 -1.9) (layer B.Fab)
       (effects (font (size 1 1) (thickness 0.15)) (justify mirror))
     )
@@
       (effects (font (size 1 1) (thickness 0.15)) (justify mirror))
     )
-    (fp_text value 1k (at 0 -1.9 90) (layer B.Fab)
+    (fp_text value 2k (at 0 -1.9 90) (layer B.Fab)
       (effects (font (size 1 1) (thickness 0.15)) (justify mirror))
     )

Commit message: refactor: use MCP6002 (and not MCP6442 which does NOT have a better performance) fix: replaced 8,2µH/0805 inductors with BLM21PG331 EMI ferrite filters
Parts:
- C19: value 4u7/16V -> 4u7
- FB1, FB2, FB3: value 8,2µH/0805 -> BLM21PG331
Changed lines of the file:
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@@
       (effects (font (size 1 1) (thickness 0.15)))
     )
-    (fp_text value 4u7/16V (at 0 2.1) (layer F.Fab)
+    (fp_text value 4u7 (at 0 2.1) (layer F.Fab)
       (effects (font (size 1 1) (thickness 0.15)))
     )
@@
       (effects (font (size 1 1) (thickness 0.15)))
     )
-    (fp_text value 8,2µH/0805 (at 0 2.1) (layer F.Fab)
+    (fp_text value BLM21PG331 (at 0 2.1) (layer F.Fab)
       (effects (font (size 1 1) (thickness 0.15)))
     )
@@
       (effects (font (size 1 1) (thickness 0.15)))
     )
-    (fp_text value 8,2µH/0805 (at 0 2.1) (layer F.Fab)
+    (fp_text value BLM21PG331 (at 0 2.1) (layer F.Fab)
       (effects (font (size 1 1) (thickness 0.15)))
     )
@@
       (effects (font (size 1 1) (thickness 0.15)) (justify mirror))
     )
-    (fp_text value 8,2µH/0805 (at 0 -2.1) (layer B.Fab)
-      (effects (font (size 1 1) (thickness 0.15)) (justify mirror))
-    )
+    (fp_text value BLM21PG331 (at 0 -2.1) (layer B.Fab)
+      (effects (font (size 1 1) (thickness 0.15)) (justify mirror))
+    )

Commit message: fix: due to internal resistance of unbuffered DAC output (~15k), R8 is lowered to 2k
Parts:
- R8: value 18k -> 2k
Changed lines of the file:
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@@
       (effects (font (size 1 1) (thickness 0.15)) (justify mirror))
     )
-    (fp_text value 18k (at 0 -1.9) (layer B.Fab)
+    (fp_text value 2k (at 0 -1.9) (layer B.Fab)
       (effects (font (size 1 1) (thickness 0.15)) (justify mirror))
     )

Commit message: chore: change some resistors, caps and resonator to "DNF"
Parts:
- C5, C7: value 10n -> DNF
- R5, R6: value 10k -> DNF
Changed lines of the file:
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@@
       (effects (font (size 1 1) (thickness 0.15)) (justify mirror))
     )
-    (fp_text value 10n (at 0 -1.9 180) (layer B.Fab)
+    (fp_text value DNF (at 0 -1.9 180) (layer B.Fab)
       (effects (font (size 1 1) (thickness 0.15)) (justify mirror))
     )
@@
       (effects (font (size 1 1) (thickness 0.15)) (justify mirror))
     )
-    (fp_text value 10n (at 0 -1.9) (layer B.Fab)
+    (fp_text value DNF (at 0 -1.9) (layer B.Fab)
       (effects (font (size 1 1) (thickness 0.15)) (justify mirror))
     )
@@
       (effects (font (size 1 1) (thickness 0.15)) (justify mirror))
     )
-    (fp_text value 10k (at 0 -1.9) (layer B.Fab)
+    (fp_text value DNF (at 0 -1.9) (layer B.Fab)
       (effects (font (size 1 1) (thickness 0.15)) (justify mirror))
     )
@@
       (effects (font (size 1 1) (thickness 0.15)) (justify mirror))
     )
-    (fp_text value 10k (at 0 -1.9 180) (layer B.Fab)
-      (effects (font (size 1 1) (thickness 0.15)) (justify mirror))
-    )
+    (fp_text value DNF (at 0 -1.9 180) (layer B.Fab)
+      (effects (font (size 1 1) (thickness 0.15)) (justify mirror))
+    )
